File: touch_board.brd (EAGLE design)
At the start: 81 x 62.2 mm, 54 parts, among them IC1 PIC18F47K42-I_PT, IC2 MAX203EEWP, K1 G6K-2P, X5 Relay conn, X6 MINI-USB-UX60A-MB-5ST

Commit message: up
Connections:
- removed net N$19: IC1.44, IC2.2, SV5.7
- new net N$24: IC1.44, IC2.2, SV5.7, XT1.2
- net N$20: no longer XT1.2
Routing:
- net N$24: track 0.00 -> 180.0 mm, vias 0 -> 3
- net N$20: track 111.4 -> 38.8 mm
- net N$19: track 72.1 -> 0.00 mm, vias 3 -> 0
Changed lines of the file:
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@@
 <via x="21.336" y="55.7784" extent="1-16" drill="0.35"/>
-</signal>
-<signal name="N$19">
-<contactref element="IC2" pad="2"/>
-<contactref element="IC1" pad="44"/>
-<contactref element="SV5" pad="7"/>
-<wire x1="59.436" y1="56.5404" x2="59.436" y2="55.3212" width="0.1524" layer="1"/>
-<wire x1="53.6448" y1="62.3316" x2="59.436" y2="56.5404" width="0.1524" layer="1"/>
-<wire x1="53.6448" y1="63.0936" x2="53.6448" y2="62.3316" width="0.1524" layer="16"/>
-<wire x1="56.6928" y1="66.1416" x2="53.6448" y2="63.0936" width="0.1524" layer="16"/>
-<wire x1="64.9224" y1="66.1416" x2="56.6928" y2="66.1416" width="0.1524" layer="16"/>
-<wire x1="66.294" y1="64.77" x2="64.9224" y2="66.1416" width="0.1524" layer="16"/>
-<wire x1="66.294" y1="63.246" x2="66.294" y2="64.77" width="0.1524" layer="16"/>
-<wire x1="67.31" y1="62.23" x2="66.294" y2="63.246" width="0.1524" layer="16"/>
-<wire x1="59.436" y1="55.3212" x2="59.5" y2="55.268" width="0.1524" layer="1"/>
-<wire x1="19.6596" y1="64.1604" x2="19.2024" y2="64.1604" width="0.1524" layer="1"/>
-<wire x1="21.0312" y1="65.532" x2="19.6596" y2="64.1604" width="0.1524" layer="1"/>
-<wire x1="21.0312" y1="67.5132" x2="21.0312" y2="65.532" width="0.1524" layer="16"/>
-<wire x1="27.2796" y1="73.7616" x2="21.0312" y2="67.5132" width="0.1524" layer="16"/>
-<wire x1="32.766" y1="73.7616" x2="27.2796" y2="73.7616" width="0.1524" layer="16"/>
-<wire x1="42.672" y1="63.8556" x2="32.766" y2="73.7616" width="0.1524" layer="16"/>
-<wire x1="46.7868" y1="63.8556" x2="42.672" y2="63.8556" width="0.1524" layer="16"/>
-<wire x1="52.1208" y1="63.8556" x2="46.7868" y2="63.8556" width="0.1524" layer="1"/>
-<wire x1="53.6448" y1="62.3316" x2="52.1208" y2="63.8556" width="0.1524" layer="1"/>
-<wire x1="19.2024" y1="64.1604" x2="19.1008" y2="64.135" width="0.1524" layer="1"/>
-<via x="53.6448" y="62.3316" extent="1-16" drill="0.35"/>
-<via x="21.0312" y="65.532" extent="1-16" drill="0.35"/>
-<via x="46.7868" y="63.8556" extent="1-16" drill="0.35"/>
 </signal>
 <signal name="N$20">
 <contactref element="IC2" pad="1"/>
 <contactref element="SERIAL/ICSP" pad="1"/>
-<contactref element="XT1" pad="2"/>
 <wire x1="18.5928" y1="65.3796" x2="19.05" y2="65.3796" width="0.1524" layer="1"/>
 <wire x1="16.9164" y1="63.7032" x2="18.5928" y2="65.3796" width="0.1524" layer="1"/>
@@
 <wire x1="19.05" y1="65.3796" x2="19.1008" y2="65.405" width="0.1524" layer="1"/>
 <wire x1="22.86" y1="30.3276" x2="22.9" y2="30.27" width="0.1524" layer="1"/>
-<wire x1="82.1436" y1="28.4988" x2="82.4484" y2="28.4988" width="0.1524" layer="1"/>
-<wire x1="77.5716" y1="23.9268" x2="82.1436" y2="28.4988" width="0.1524" layer="1"/>
-<wire x1="71.3232" y1="23.9268" x2="77.5716" y2="23.9268" width="0.1524" layer="1"/>
-<wire x1="71.1708" y1="23.7744" x2="71.3232" y2="23.9268" width="0.1524" layer="1"/>
-<wire x1="71.1708" y1="22.098" x2="71.1708" y2="23.7744" width="0.1524" layer="1"/>
-<wire x1="68.2752" y1="19.2024" x2="71.1708" y2="22.098" width="0.1524" layer="1"/>
-<wire x1="28.0416" y1="19.2024" x2="68.2752" y2="19.2024" width="0.1524" layer="1"/>
-<wire x1="23.0124" y1="24.2316" x2="28.0416" y2="19.2024" width="0.1524" layer="1"/>
-<wire x1="23.0124" y1="30.1752" x2="23.0124" y2="24.2316" width="0.1524" layer="1"/>
-<wire x1="82.4484" y1="28.4988" x2="82.55" y2="28.575" width="0.1524" layer="1"/>
-<wire x1="23.0124" y1="30.1752" x2="22.9" y2="30.27" width="0.1524" layer="1"/>
 </signal>
 <signal name="N$21">
@@
 <via x="35.9664" y="19.812" extent="1-16" drill="0.35"/>
 </signal>
+<signal name="N$24">
+<contactref element="XT1" pad="2"/>
+<contactref element="IC2" pad="2"/>
+<contactref element="IC1" pad="44"/>
+<contactref element="SV5" pad="7"/>
+<wire x1="59.436" y1="56.5404" x2="59.436" y2="55.3212" width="0.1524" layer="1"/>
+<wire x1="53.6448" y1="62.3316" x2="59.436" y2="56.5404" width="0.1524" layer="1"/>
+<wire x1="53.6448" y1="63.0936" x2="53.6448" y2="62.3316" width="0.1524" layer="16"/>
+<wire x1="56.6928" y1="66.1416" x2="53.6448" y2="63.0936" width="0.1524" layer="16"/>
+<wire x1="64.9224" y1="66.1416" x2="56.6928" y2="66.1416" width="0.1524" layer="16"/>
+<wire x1="66.294" y1="64.77" x2="64.9224" y2="66.1416" width="0.1524" layer="16"/>
+<wire x1="66.294" y1="63.246" x2="66.294" y2="64.77" width="0.1524" layer="16"/>
+<wire x1="67.31" y1="62.23" x2="66.294" y2="63.246" width="0.1524" layer="16"/>
+<wire x1="59.436" y1="55.3212" x2="59.5" y2="55.268" width="0.1524" layer="1"/>
+<wire x1="19.6596" y1="64.1604" x2="19.2024" y2="64.1604" width="0.1524" layer="1"/>
+<wire x1="21.0312" y1="65.532" x2="19.6596" y2="64.1604" width="0.1524" layer="1"/>
+<wire x1="21.0312" y1="67.5132" x2="21.0312" y2="65.532" width="0.1524" layer="16"/>
+<wire x1="27.2796" y1="73.7616" x2="21.0312" y2="67.5132" width="0.1524" layer="16"/>
+<wire x1="32.766" y1="73.7616" x2="27.2796" y2="73.7616" width="0.1524" layer="16"/>
+<wire x1="42.672" y1="63.8556" x2="34.29" y2="72.2376" width="0.1524" layer="16"/>
+<wire x1="34.29" y1="72.2376" x2="32.766" y2="73.7616" width="0.1524" layer="16"/>
+<wire x1="46.7868" y1="63.8556" x2="42.672" y2="63.8556" width="0.1524" layer="16"/>
+<wire x1="52.1208" y1="63.8556" x2="46.7868" y2="63.8556" width="0.1524" layer="1"/>
+<wire x1="53.6448" y1="62.3316" x2="52.1208" y2="63.8556" width="0.1524" layer="1"/>
+<wire x1="19.2024" y1="64.1604" x2="19.1008" y2="64.135" width="0.1524" layer="1"/>
+<via x="53.6448" y="62.3316" extent="1-16" drill="0.35"/>
+<via x="21.0312" y="65.532" extent="1-16" drill="0.35"/>
+<via x="46.7868" y="63.8556" extent="1-16" drill="0.35"/>
+<wire x1="82.6008" y1="35.9664" x2="82.6008" y2="28.6512" width="0.1524" layer="16"/>
+<wire x1="91.5924" y1="44.958" x2="82.6008" y2="35.9664" width="0.1524" layer="16"/>
+<wire x1="91.5924" y1="73.6092" x2="91.5924" y2="44.958" width="0.1524" layer="16"/>
+<wire x1="90.3732" y1="74.8284" x2="91.5924" y2="73.6092" width="0.1524" layer="16"/>
+<wire x1="55.4736" y1="74.8284" x2="90.3732" y2="74.8284" width="0.1524" layer="16"/>
+<wire x1="53.7972" y1="73.152" x2="55.4736" y2="74.8284" width="0.1524" layer="16"/>
+<wire x1="36.576" y1="73.152" x2="53.7972" y2="73.152" width="0.1524" layer="16"/>
+<wire x1="36.2712" y1="73.4568" x2="36.576" y2="73.152" width="0.1524" layer="16"/>
+<wire x1="35.5092" y1="73.4568" x2="36.2712" y2="73.4568" width="0.1524" layer="16"/>
+<wire x1="34.29" y1="72.2376" x2="35.5092" y2="73.4568" width="0.1524" layer="16"/>
+<wire x1="82.6008" y1="28.6512" x2="82.55" y2="28.575" width="0.1524" layer="16"/>
+</signal>
 </signals>
