File: touch_board.sch (EAGLE design)
At the start: 54 parts, among them IC1 PIC18F47K42-I_PT, IC2 MAX203EEWP, K1 G6K-2P, X5 Relay conn, X6 MINI-USB-UX60A-MB-5ST

Commit message: up
Connections:
- removed net N$19: IC1.RC6, IC2G$1.T1IN, SV5.7
- new net N$24: IC1.RC6, IC2G$1.T1IN, SV5.7, XT1.C
- net N$20: no longer XT1.C
Changed lines of the file:
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@@
-</segment>
-</net>
-<net name="N$19" class="0">
-<segment>
-<pinref part="IC2" gate="G$1" pin="T1IN"/>
-<wire x1="-30.48" y1="25.4" x2="-40.64" y2="25.4" width="0.1524" layer="91"/>
-<wire x1="-40.64" y1="25.4" x2="-40.64" y2="83.82" width="0.1524" layer="91"/>
-<wire x1="-40.64" y1="83.82" x2="60.96" y2="83.82" width="0.1524" layer="91"/>
-<pinref part="IC1" gate="G$1" pin="RC6"/>
-<wire x1="60.96" y1="83.82" x2="60.96" y2="66.04" width="0.1524" layer="91"/>
-<junction x="-30.48" y="25.4"/>
-<junction x="60.96" y="66.04"/>
-<wire x1="60.96" y1="83.82" x2="60.96" y2="106.68" width="0.1524" layer="91"/>
-<wire x1="60.96" y1="106.68" x2="180.34" y2="106.68" width="0.1524" layer="91"/>
-<wire x1="180.34" y1="106.68" x2="180.34" y2="66.04" width="0.1524" layer="91"/>
-<pinref part="SV5" gate="G$1" pin="7"/>
-<wire x1="180.34" y1="66.04" x2="172.72" y2="66.04" width="0.1524" layer="91"/>
-<junction x="60.96" y="83.82"/>
-<junction x="172.72" y="66.04"/>
 </segment>
 </net>
@@
 <wire x1="-30.48" y1="22.86" x2="-40.64" y2="22.86" width="0.1524" layer="91"/>
 <wire x1="-40.64" y1="22.86" x2="-40.64" y2="5.08" width="0.1524" layer="91"/>
-<wire x1="-40.64" y1="5.08" x2="-20.32" y2="5.08" width="0.1524" layer="91"/>
 <junction x="-30.48" y="22.86"/>
-<wire x1="-20.32" y1="5.08" x2="20.32" y2="5.08" width="0.1524" layer="91"/>
+<wire x1="-40.64" y1="5.08" x2="20.32" y2="5.08" width="0.1524" layer="91"/>
 <wire x1="20.32" y1="-35.56" x2="20.32" y2="5.08" width="0.1524" layer="91"/>
 <wire x1="20.32" y1="-35.56" x2="7.62" y2="-35.56" width="0.1524" layer="91"/>
@@
 <wire x1="7.62" y1="-55.88" x2="20.32" y2="-55.88" width="0.1524" layer="91"/>
 <junction x="20.32" y="-55.88"/>
-<pinref part="XT1" gate="A" pin="C"/>
-<wire x1="-35.56" y1="-22.86" x2="-20.32" y2="-22.86" width="0.1524" layer="91"/>
-<wire x1="-20.32" y1="-22.86" x2="-20.32" y2="5.08" width="0.1524" layer="91"/>
-<junction x="-20.32" y="5.08"/>
-<junction x="-35.56" y="-22.86"/>
 </segment>
 </net>
@@
 </segment>
 </net>
+<net name="N$24" class="0">
+<segment>
+<pinref part="XT1" gate="A" pin="C"/>
+<junction x="-35.56" y="-22.86"/>
+<wire x1="-35.56" y1="-22.86" x2="-20.32" y2="-22.86" width="0.1524" layer="91"/>
+<wire x1="-20.32" y1="-22.86" x2="-20.32" y2="0" width="0.1524" layer="91"/>
+<wire x1="-20.32" y1="0" x2="-48.26" y2="0" width="0.1524" layer="91"/>
+<pinref part="IC2" gate="G$1" pin="T1IN"/>
+<wire x1="-30.48" y1="25.4" x2="-40.64" y2="25.4" width="0.1524" layer="91"/>
+<wire x1="-40.64" y1="25.4" x2="-40.64" y2="33.02" width="0.1524" layer="91"/>
+<wire x1="-40.64" y1="33.02" x2="-40.64" y2="83.82" width="0.1524" layer="91"/>
+<wire x1="-40.64" y1="83.82" x2="60.96" y2="83.82" width="0.1524" layer="91"/>
+<pinref part="IC1" gate="G$1" pin="RC6"/>
+<wire x1="60.96" y1="83.82" x2="60.96" y2="66.04" width="0.1524" layer="91"/>
+<junction x="-30.48" y="25.4"/>
+<junction x="60.96" y="66.04"/>
+<wire x1="60.96" y1="83.82" x2="60.96" y2="106.68" width="0.1524" layer="91"/>
+<wire x1="60.96" y1="106.68" x2="180.34" y2="106.68" width="0.1524" layer="91"/>
+<wire x1="180.34" y1="106.68" x2="180.34" y2="66.04" width="0.1524" layer="91"/>
+<pinref part="SV5" gate="G$1" pin="7"/>
+<wire x1="180.34" y1="66.04" x2="172.72" y2="66.04" width="0.1524" layer="91"/>
+<junction x="60.96" y="83.82"/>
+<junction x="172.72" y="66.04"/>
+<wire x1="-48.26" y1="0" x2="-48.26" y2="33.02" width="0.1524" layer="91"/>
+<wire x1="-48.26" y1="33.02" x2="-40.64" y2="33.02" width="0.1524" layer="91"/>
+<junction x="-40.64" y="33.02"/>
+</segment>
+</net>

Commit message: up
Other:
- note added: "Really 47Q43"
Changed lines of the file:
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@@
 <sheet>
 <plain>
+<text x="91.44" y="58.42" size="1.778" layer="91">Really 47Q43</text>
+<text x="68.58" y="22.86" size="1.778" layer="91">Really 47Q43</text>
+<text x="66.04" y="50.8" size="1.778" layer="91">Really 47Q43</text>
 </plain>
 <instances>
